Commit message: add the eai lidar

File: src/spark/spark_description/robots/spark.urdf.xacro (robot description, xacro)
@@ -7,6 +7,8 @@
 <robot name="spark" xmlns:xacro="http://ros.org/wiki/xacro">
 	<xacro:arg name="camera_types" default="astrapro"/>
+	<xacro:arg name="lidar_type_tel"	default="3iroboticslidar2"/>
   	<xacro:include filename="$(find spark_description)/urdf/spark_340.urdf.xacro">
 		<xacro:arg name="camera_types"	value="$(arg camera_types)"/>
+		<xacro:arg name="lidar_type_tel"	value="$(arg lidar_type_tel)"/>
 	</xacro:include>
 </robot>

File: src/spark/spark_description/urdf/spark_340.urdf.xacro (robot description, xacro)
@@ -8,7 +8,14 @@
   	<xacro:arg name="camera_types"	default="astrapro"/>
 	<xacro:property name="camera"	value="$(arg camera_types)"/>
+  	<xacro:arg name="lidar_type_tel"	default="astrapro"/>
+	<xacro:property name="lidar"	value="$(arg lidar_type_tel)"/>
   	<xacro:include filename="$(find spark_description)/urdf/base/spark_base.urdf"/>
   	<xacro:include filename="$(find spark_description)/urdf/stack/spark_stack.urdf"/>
-	<xacro:include filename="$(find spark_description)/urdf/sensors/spark_lidar.urdf"/>
+	<xacro:if value="${lidar == 'ydlidar_g2'}">
+		<xacro:include filename="$(find ydlidar_g2)/urdf/ydlidar.urdf" />
+	</xacro:if>
+	<xacro:if value="${lidar == '3iroboticslidar2'}">
+		<xacro:include filename="$(find spark_description)/urdf/sensors/spark_lidar.urdf"/>
+	</xacro:if>
 	<xacro:if value="${camera == 'astrapro' or camera == 'astra'}">
 		<xacro:include filename="$(find spark_description)/urdf/sensors/spark_$(arg camera_types).urdf"/>

Commit message: 加入机械臂相关选择。修改摄像头设备参数

File: src/spark/spark_description/robots/spark.urdf.xacro (robot description, xacro)
@@ -6,8 +6,8 @@
 -->
 <robot name="spark" xmlns:xacro="http://ros.org/wiki/xacro">
-	<xacro:arg name="camera_types" default="astrapro"/>
+	<xacro:arg name="camera_type_tel" default="astrapro"/>
 	<xacro:arg name="lidar_type_tel"	default="3iroboticslidar2"/>
   	<xacro:include filename="$(find spark_description)/urdf/spark_340.urdf.xacro">
-		<xacro:arg name="camera_types"	value="$(arg camera_types)"/>
+		<xacro:arg name="camera_type_tel"	value="$(arg camera_type_tel)"/>
 		<xacro:arg name="lidar_type_tel"	value="$(arg lidar_type_tel)"/>
 	</xacro:include>

File: src/spark/spark_description/urdf/spark_340.urdf.xacro (robot description, xacro)
@@ -6,6 +6,10 @@
 -->
 <robot name="spark" xmlns:xacro="http://ros.org/wiki/xacro">
-  	<xacro:arg name="camera_types"	default="astrapro"/>
-	<xacro:property name="camera"	value="$(arg camera_types)"/>
+	<xacro:arg name="enable_arm_tel"	default="false"/>
+	<xacro:property name="enable_arm"	value="$(arg enable_arm_tel)"/>
+	<xacro:arg name="arm_type_tel"	default="uarm"/>
+	<xacro:property name="robot_arm_type"	value="$(arg arm_type_tel)"/>
+  	<xacro:arg name="camera_type_tel"	default="astrapro"/>
+	<xacro:property name="camera"	value="$(arg camera_type_tel)"/>
   	<xacro:arg name="lidar_type_tel"	default="astrapro"/>
 	<xacro:property name="lidar"	value="$(arg lidar_type_tel)"/>
@@ -22,8 +26,16 @@
 	</xacro:if>
 	<xacro:if value="${camera == 'astrapro' or camera == 'astra'}">
-		<xacro:include filename="$(find spark_description)/urdf/sensors/spark_$(arg camera_types).urdf"/>
+		<xacro:include filename="$(find spark_description)/urdf/sensors/spark_$(arg camera_type_tel).urdf"/>
 	</xacro:if>
 	<xacro:if value="${camera == 'd435'}">
 		<xacro:include filename="$(find spark_description)/urdf/sensors/spark_d435.urdf.xacro"/>
 	</xacro:if>
+	<xacro:if value="${enable_arm == 'true'}">
+		<xacro:if value="${robot_arm_type == 'sagittarius_arm'}">
+  			<xacro:include filename="$(find sagittarius_descriptions)/urdf/spark_sagittarius_descriptions.urdf"/>
+		</xacro:if>
+        	<xacro:if value="${robot_arm_type == 'uarm'}">
+  			<xacro:include filename="$(find swiftpro)/urdf/spark_pro_model.xacro"/>
+		</xacro:if>
+	</xacro:if>
 </robot>

File: src/spark_driver/lidar/ydlidar_g2/urdf/ydlidar.urdf (robot description, URDF)
Before this commit: robot ydlidar_g2, 3 links, 3 joints
Links:
- removed link lidar_bottom_screw_frame
Joints:
- removed joint lidar_joint
- joint lidar_link_joint: parent lidar_bottom_screw_frame -> base_link
